File: kicad/small-lm399.kicad_pcb (KiCad board)
At the start: 2 copper layers, 25.4 x 38.1 mm, 17 parts, among them P1 CONN_1X1, P2 CONN_1X1, P3 CONN_1X1, P4 CONN_1X1, P5 CONN_1X1, P6 CONN_2X1, P7 CONN_1X1, P8 CONN_1X1, U1 LM399, U2 OP07

Commit message: adding schematic
Parts:
- removed the C1 at (302.3, 63.5)
- removed the C2 at (304.8, 54.6)
- removed the C3 at (312.4, 63.5)
- removed P1, P2, P3, P4, P5, P7, P8: CONN_1X1, SIL-1
- removed P6: CONN_2X1, SIL-2
- removed the R1 at (318.1, 48.3)
- removed the R2 at (318.8, 61.0)
- removed the R3 at (302.3, 58.4)
- removed the U2 at (307.3, 58.4)
- added 4455-N2-5: Val**, 4455-N2-5, F.Cu at (-172.1, 245.1)
- added 4455-N2-5: Val**, 4455-N2-5, F.Cu at (-281.3, 111.1)
- added 4455-N2-5: Val**, 4455-N2-5, F.Cu at (-152.4, 123.2)
- added 4455-N2-5: Val**, 4455-N2-5, F.Cu at (-130.8, 110.5)
- added 4455-N2-5: Val**, 4455-N2-5, F.Cu at (-379.7, 123.2)
- added 4455-N2-5: Val**, 4455-N2-5, F.Cu at (-358.1, 110.5)
- added 4455-N2-5: Val**, 4455-N2-5, F.Cu at (-207.0, 111.8)
- added 4455-N2-5: Val**, 4455-N2-5, F.Cu at (-228.6, 124.5)
- added 4455-N2-5: Val**, 4455-N2-5, F.Cu at (-228.6, 14.0)
- added 4455-N2-5: Val**, 4455-N2-5, F.Cu at (-250.2, 26.7)
- added 4455-N2-5: Val**, 4455-N2-5, F.Cu at (-87.6, 43.2)
- added 4455-N2-5: Val**, 4455-N2-5, F.Cu at (-150.5, 232.4)
- added 4455-N2-5: Val**, 4455-N2-5, F.Cu at (-66.0, 30.5)
- added 4455-N2-5: Val**, 4455-N2-5, F.Cu at (120.7, 368.3)
- added 4455-N2-5: Val**, 4455-N2-5, F.Cu at (142.2, 381.0)
- added 4455-N2-5: Val**, 4455-N2-5, F.Cu at (91.4, 381.0)
- added 4455-N2-5: Val**, 4455-N2-5, F.Cu at (69.8, 368.3)
- added 4455-N2-5: Val**, 4455-N2-5, F.Cu at (99.1, 449.6)
- added 4455-N2-5: Val**, 4455-N2-5, F.Cu at (120.7, 462.3)
- added 4455-N2-5: Val**, 4455-N2-5, F.Cu at (48.3, 449.6)
- added 4455-N2-5: Val**, 4455-N2-5, F.Cu at (69.8, 462.3)
- added 4455-N2-5: Val**, 4455-N2-5, F.Cu at (337.8, 452.1)
- added 4455-N2-5: Val**, 4455-N2-5, F.Cu at (-215.3, 233.0)
- added 4455-N2-5: Val**, 4455-N2-5, F.Cu at (359.4, 464.8)
- added 4455-N2-5: Val**, 4455-N2-5, F.Cu at (360.7, 388.6)
- added 4455-N2-5: Val**, 4455-N2-5, F.Cu at (339.1, 375.9)
- added 4455-N2-5: Val**, 4455-N2-5, F.Cu at (-236.9, 245.7)
- added 4455-N2-5: Val**, 4455-N2-5, F.Cu at (-302.9, 245.7)
- added 4455-N2-5: Val**, 4455-N2-5, F.Cu at (-281.3, 233.0)
- added 4455-N2-5: Val**, 4455-N2-5, F.Cu at (-281.3, 174.0)
- added 4455-N2-5: Val**, 4455-N2-5, F.Cu at (-302.9, 186.7)
- added 4455-N2-5: Val**, 4455-N2-5, F.Cu at (-302.9, 123.8)
- added C1: 0.1uF, CERCAP_2_059A, F.Cu at (-162.6, 245.7)
- added C1: 0.1uF, CERCAP_2_059A, F.Cu at (-227.3, 246.4)
- added C1: 0.1uF, CERCAP_2_059A, F.Cu at (-143.5, 123.2)
- added C2: 0.1uF, CERCAP_2_059A, F.Cu at (-153.7, 245.7)
- added C2: 0.1uF, CERCAP_2_059A, F.Cu at (-218.4, 246.4)
- added C2: 0.1uF, CERCAP_2_059A, F.Cu at (-134.6, 123.2)
- added C3: 10nF, CERCAP_2_059A, F.Cu at (-129.5, 245.7)
- added C3: 10nF, CERCAP_2_059A, F.Cu at (-194.3, 246.4)
- added C3: 10nF, CERCAP_2_059A, F.Cu at (-110.5, 123.2)
- added H***: Val**, Via_016, F.Cu at (-174.0, 237.5)
- added H***: Val**, hole_M3_2, F.Cu at (-261.0, 257.2)
- added H***: Val**, Via_016, F.Cu at (-174.0, 262.3)
- added H***: Val**, Via_016, F.Cu at (-174.0, 264.2)
- added H***: Val**, Via_016, F.Cu at (-174.0, 266.1)
- added H***: Val**, Via_016, F.Cu at (-174.0, 268.0)
- added H***: Val**, Via_016, F.Cu at (-174.0, 269.9)
- added H***: Val**, Via_016, F.Cu at (-174.0, 271.8)
- added H***: Val**, Via_016, F.Cu at (-174.0, 273.7)
- added H***: Val**, Via_016, F.Cu at (-173.4, 275.0)
- added H***: Val**, Via_016, F.Cu at (-172.7, 276.2)
- added H***: Val**, Via_016, F.Cu at (-171.4, 276.9)
- added H***: Val**, hole_M3_2, F.Cu at (-301.6, 234.3)
- added H***: Val**, Via_016, F.Cu at (-170.2, 277.5)
- added H***: Val**, Via_016, F.Cu at (-168.3, 277.5)
- added H***: Val**, Via_016, F.Cu at (-166.4, 277.5)
- added H***: Val**, Via_016, F.Cu at (-164.5, 277.5)
- added H***: Val**, Via_016, F.Cu at (-162.6, 277.5)
- added H***: Val**, Via_016, F.Cu at (-160.7, 277.5)
- added H***: Val**, Via_016, F.Cu at (-158.8, 277.5)
- added H***: Val**, Via_016, F.Cu at (-156.8, 277.5)
- added H***: Val**, Via_016, F.Cu at (-154.9, 277.5)
- added H***: Val**, Via_016, F.Cu at (-153.0, 277.5)
- added H***: Val**, hole_M3_2, F.Cu at (-261.0, 234.3)
- added H***: Val**, Via_016, F.Cu at (-151.3, 277.5)
- added H***: Val**, Via_016, F.Cu at (-149.7, 277.5)
- added H***: Val**, Via_016, F.Cu at (-148.0, 277.5)
- added H***: Val**, Via_016, F.Cu at (-146.1, 277.5)
- added H***: Val**, Via_016, F.Cu at (-144.1, 277.5)
- added H***: Val**, Via_016, F.Cu at (-142.2, 277.5)
- added H***: Val**, Via_016, F.Cu at (-140.3, 277.5)
- added H***: Val**, Via_016, F.Cu at (-138.4, 277.5)
- added H***: Val**, Via_016, F.Cu at (-136.5, 277.5)
- added H***: Val**, Via_016, F.Cu at (-134.6, 277.5)
- added H***: Val**, hole_M3_2, F.Cu at (-301.6, 257.2)
- added H***: Val**, Via_016, F.Cu at (-132.7, 277.5)
- added H***: Val**, Via_016, F.Cu at (-130.8, 277.5)
- added H***: Val**, Via_016, F.Cu at (-129.5, 276.9)
- added H***: Val**, Via_016, F.Cu at (-127.6, 275.0)
- added H***: Val**, Via_016, F.Cu at (-127.0, 273.7)
- added H***: Val**, Via_016, F.Cu at (-128.3, 276.2)
- added H***: Val**, Via_016, F.Cu at (-127.0, 271.8)
- added H***: Val**, Via_016, F.Cu at (-127.0, 269.9)
- added H***: Val**, Via_016, F.Cu at (-127.0, 268.0)
- added H***: Val**, Via_016, F.Cu at (-127.0, 266.1)
- added H***: Val**, hole_M3_2, F.Cu at (-301.6, 198.1)
- added H***: Val**, Via_016, F.Cu at (-127.0, 264.2)
- added H***: Val**, Via_016, F.Cu at (-127.0, 262.3)
- added H***: Val**, Via_016, F.Cu at (-127.0, 260.4)
- added H***: Val**, Via_016, F.Cu at (-127.0, 252.7)
- added H***: Val**, Via_016, F.Cu at (-127.0, 250.8)
- added H***: Val**, Via_016, F.Cu at (-127.0, 248.9)
- added H***: Val**, Via_016, F.Cu at (-127.0, 247.0)
- added H***: Val**, Via_016, F.Cu at (-127.0, 245.1)
- added H***: Val**, Via_016, F.Cu at (-127.0, 243.2)
- added H***: Val**, Via_016, F.Cu at (-127.0, 241.3)
- added H***: Val**, hole_M3_2, F.Cu at (-261.0, 175.3)
- added H***: Val**, Via_016, F.Cu at (-127.0, 239.4)
- added H***: Val**, Via_016, F.Cu at (-127.0, 237.5)
- added H***: Val**, Via_016, F.Cu at (-128.9, 237.5)
- added H***: Val**, Via_016, F.Cu at (-130.8, 237.5)
- added H***: Val**, Via_016, F.Cu at (-134.0, 234.3)
- added H***: Val**, Via_016, F.Cu at (-134.0, 230.5)
- added H***: Val**, Via_016, F.Cu at (-134.0, 232.4)
- added H***: Val**, Via_016, F.Cu at (-134.0, 236.2)
- added H***: Val**, Via_016, F.Cu at (-132.7, 237.5)
- added H***: Val**, Via_016, F.Cu at (-135.9, 230.5)
- added H***: Val**, hole_M3_2, F.Cu at (-301.6, 175.3)
- added H***: Val**, Via_016, F.Cu at (-137.8, 230.5)
- added H***: Val**, Via_016, F.Cu at (-139.7, 230.5)
- added H***: Val**, Via_016, F.Cu at (-141.6, 230.5)
- added H***: Val**, Via_016, F.Cu at (-143.5, 230.5)
- added H***: Val**, Via_016, F.Cu at (-145.4, 230.5)
- added H***: Val**, Via_016, F.Cu at (-147.3, 230.5)
- added H***: Val**, Via_016, F.Cu at (-149.2, 230.5)
- added H***: Val**, Via_016, F.Cu at (-151.8, 230.5)
- added H***: Val**, Via_016, F.Cu at (-153.7, 230.5)
- added H***: Val**, Via_016, F.Cu at (-155.6, 230.5)
- added H***: Val**, hole_M3_2, F.Cu at (-261.0, 198.1)
- added H***: Val**, Via_016, F.Cu at (-157.5, 230.5)
- added H***: Val**, Via_016, F.Cu at (-159.4, 230.5)
- added H***: Val**, Via_016, F.Cu at (-161.3, 230.5)
- added H***: Val**, Via_016, F.Cu at (-163.2, 230.5)
- added H***: Val**, Via_016, F.Cu at (-167.0, 230.5)
- added H***: Val**, Via_016, F.Cu at (-165.1, 230.5)
- added H***: Val**, Via_016, F.Cu at (-128.9, 252.7)
- added H***: Val**, Via_016, F.Cu at (-128.9, 260.4)
- added H***: Val**, Via_016, F.Cu at (-130.8, 260.4)
- added H***: Val**, Via_016, F.Cu at (-130.8, 252.7)
- added H***: Val**, hole_M3_2, F.Cu at (-261.0, 135.3)
- added H***: Val**, Via_016, F.Cu at (-134.0, 256.5)
- added H***: Val**, Via_016, F.Cu at (-134.0, 254.6)
- added H***: Val**, Via_016, F.Cu at (-134.0, 258.4)
- added H***: Val**, Via_016, F.Cu at (-132.7, 259.7)
- added H***: Val**, Via_016, F.Cu at (-132.7, 253.4)
- added H***: Val**, Via_016, F.Cu at (-167.0, 232.4)
- added H***: Val**, Via_016, F.Cu at (-167.0, 234.3)
- added H***: Val**, Via_016, F.Cu at (-172.1, 237.5)
- added H***: Val**, Via_016, F.Cu at (-170.2, 237.5)
- added H***: Val**, Via_016, F.Cu at (-168.3, 237.5)
- added H***: Val**, hole_M3_2, F.Cu at (-301.6, 112.4)
- added H***: Val**, Via_016, F.Cu at (-167.0, 236.2)
- added H***: Val**, Via_016, F.Cu at (-137.8, 271.8)
- added H***: Val**, Via_016, F.Cu at (-135.9, 269.2)
- added H***: Val**, Via_016, F.Cu at (-134.6, 270.5)
- added H***: Val**, Via_016, F.Cu at (-135.9, 271.8)
- added H***: Val**, Via_016, F.Cu at (-139.7, 271.1)
- added H***: Val**, Via_016, F.Cu at (-142.2, 266.7)
- added H***: Val**, Via_016, F.Cu at (-137.8, 268.6)
- added H***: Val**, Via_016, F.Cu at (-139.1, 267.3)
- added H***: Val**, Via_016, F.Cu at (-139.7, 265.4)
- added H***: Val**, hole_M3_2, F.Cu at (-130.2, 256.5)
- added H***: Val**, hole_M3_2, F.Cu at (-261.0, 112.4)
- added H***: Val**, Via_016, F.Cu at (-141.0, 269.9)
- added H***: Val**, Via_016, F.Cu at (-141.6, 268.6)
- added H***: Val**, Via_016, F.Cu at (-139.7, 263.5)
- added H***: Val**, Via_016, F.Cu at (-139.7, 261.6)
- added H***: Val**, Via_016, F.Cu at (-140.3, 259.7)
- added H***: Val**, Via_016, F.Cu at (-141.6, 258.4)
- added H***: Val**, Via_016, F.Cu at (-142.9, 257.2)
- added H***: Val**, Via_016, F.Cu at (-144.1, 255.9)
- added H***: Val**, Via_016, F.Cu at (-146.1, 255.3)
- added H***: Val**, Via_016, F.Cu at (-148.0, 254.6)
- added H***: Val**, hole_M3_2, F.Cu at (-301.6, 135.3)
- added H***: Val**, Via_016, F.Cu at (-149.7, 254.6)
- added H***: Val**, Via_016, F.Cu at (-151.3, 254.6)
- added H***: Val**, Via_016, F.Cu at (-153.7, 255.3)
- added H***: Val**, Via_016, F.Cu at (-155.6, 255.3)
- added H***: Val**, hole_M3_2, F.Cu at (-110.5, 134.6)
- added H***: Val**, hole_M3_2, F.Cu at (-151.1, 111.8)
- added H***: Val**, hole_M3_2, F.Cu at (-110.5, 111.8)
- added H***: Val**, hole_M3_2, F.Cu at (-151.1, 134.6)
- added H***: Val**, hole_M3_2, F.Cu at (-337.8, 134.6)
- added H***: Val**, hole_M3_2, F.Cu at (-378.5, 111.8)
- added H***: Val**, hole_M3_2, F.Cu at (-337.8, 111.8)
- added H***: Val**, hole_M3_2, F.Cu at (-378.5, 134.6)
- added H***: Val**, hole_M3_2, F.Cu at (-170.8, 233.7)
- added H***: Val**, hole_M3_2, F.Cu at (-227.3, 135.9)
- added H***: Val**, hole_M3_2, F.Cu at (-186.7, 113.0)
- added H***: Val**, hole_M3_2, F.Cu at (-227.3, 113.0)
- added H***: Val**, hole_M3_2, F.Cu at (-186.7, 135.9)
- added H***: Val**, hole_M3_2, F.Cu at (-248.9, 38.1)
- added H***: Val**, hole_M3_2, F.Cu at (-208.3, 15.2)
- added H***: Val**, hole_M3_2, F.Cu at (-248.9, 15.2)
- added H***: Val**, hole_M3_2, F.Cu at (-208.3, 38.1)
- added H***: Val**, hole_M3_2, F.Cu at (-45.7, 54.6)
- added H***: Val**, hole_M3_2, F.Cu at (-86.4, 31.8)
- added H***: Val**, hole_M3_2, F.Cu at (-130.2, 233.7)
- added H***: Val**, hole_M3_2, F.Cu at (-45.7, 31.8)
- added H***: Val**, hole_M3_2, F.Cu at (-86.4, 54.6)
- added H***: Val**, hole_M3_2, F.Cu at (283.2, 435.6)
- added H***: Val**, hole_M3_2, F.Cu at (191.8, 458.5)
- added H***: Val**, hole_M3_2, F.Cu at (232.4, 435.6)
- added H***: Val**, hole_M3_2, F.Cu at (191.8, 435.6)
- added H***: Val**, hole_M3_2, F.Cu at (232.4, 458.5)
- added H***: Val**, hole_M3_2, F.Cu at (242.6, 458.5)
- added H***: Val**, hole_M3_2, F.Cu at (242.6, 435.6)
- added H***: Val**, hole_M3_2, F.Cu at (283.2, 458.5)
- added H***: Val**, hole_M3_2, F.Cu at (-170.8, 256.5)
- added H***: Val**, hole_M3_2, F.Cu at (232.4, 367.0)
- added H***: Val**, hole_M3_2, F.Cu at (191.8, 389.9)
- added H***: Val**, hole_M3_2, F.Cu at (232.4, 389.9)
- added H***: Val**, hole_M3_2, F.Cu at (191.8, 367.0)
- added H***: Val**, hole_M3_2, F.Cu at (242.6, 367.0)
- added H***: Val**, hole_M3_2, F.Cu at (283.2, 389.9)
- added H***: Val**, hole_M3_2, F.Cu at (242.6, 389.9)
- added H***: Val**, hole_M3_2, F.Cu at (283.2, 367.0)
- added H***: Val**, hole_M3_2, F.Cu at (141.0, 369.6)
- added H***: Val**, hole_M3_2, F.Cu at (100.3, 392.4)
- added H***: Val**, hole_M3_2, F.Cu at (-235.6, 257.2)
- added H***: Val**, hole_M3_2, F.Cu at (141.0, 392.4)
- added H***: Val**, hole_M3_2, F.Cu at (100.3, 369.6)
- added H***: Val**, hole_M3_2, F.Cu at (49.5, 369.6)
- added H***: Val**, hole_M3_2, F.Cu at (90.2, 392.4)
- added H***: Val**, hole_M3_2, F.Cu at (49.5, 392.4)
- added H***: Val**, hole_M3_2, F.Cu at (90.2, 369.6)
- added H***: Val**, hole_M3_2, F.Cu at (141.0, 461.0)
- added H***: Val**, hole_M3_2, F.Cu at (100.3, 438.1)
- added H***: Val**, hole_M3_2, F.Cu at (141.0, 438.1)
- added H***: Val**, hole_M3_2, F.Cu at (100.3, 461.0)
- added H***: Val**, hole_M3_2, F.Cu at (-194.9, 234.3)
- added H***: Val**, hole_M3_2, F.Cu at (90.2, 461.0)
- added H***: Val**, hole_M3_2, F.Cu at (49.5, 438.1)
- added H***: Val**, hole_M3_2, F.Cu at (90.2, 438.1)
- added H***: Val**, hole_M3_2, F.Cu at (49.5, 461.0)
- added H***: Val**, hole_M3_2, F.Cu at (379.7, 463.6)
- added H***: Val**, hole_M3_2, F.Cu at (339.1, 440.7)
- added H***: Val**, hole_M3_2, F.Cu at (379.7, 440.7)
- added H***: Val**, hole_M3_2, F.Cu at (339.1, 463.6)
- added H***: Val**, hole_M3_2, F.Cu at (340.4, 387.4)
- added H***: Val**, hole_M3_2, F.Cu at (381.0, 364.5)
- added H***: Val**, hole_M3_2, F.Cu at (-235.6, 234.3)
- added H***: Val**, hole_M3_2, F.Cu at (340.4, 364.5)
- added H***: Val**, hole_M3_2, F.Cu at (381.0, 387.4)
- added H***: Val**, Via_016, F.Cu at (-174.0, 239.4)
- added H***: Val**, Via_016, F.Cu at (-174.0, 241.3)
- added H***: Val**, Via_016, F.Cu at (-174.0, 243.2)
- added H***: Val**, Via_016, F.Cu at (-174.0, 245.1)
- added H***: Val**, Via_016, F.Cu at (-174.0, 247.0)
- added H***: Val**, Via_016, F.Cu at (-174.0, 248.9)
- added H***: Val**, Via_016, F.Cu at (-174.0, 250.8)
- added H***: Val**, Via_016, F.Cu at (-174.0, 252.7)
- added H***: Val**, hole_M3_2, F.Cu at (-194.9, 257.2)
- added H***: Val**, Via_016, F.Cu at (-172.1, 252.7)
- added H***: Val**, Via_016, F.Cu at (-170.2, 252.7)
- added H***: Val**, Via_016, F.Cu at (-168.3, 253.4)
- added H***: Val**, Via_016, F.Cu at (-167.0, 254.6)
- added H***: Val**, Via_016, F.Cu at (-167.0, 256.5)
- added H***: Val**, Via_016, F.Cu at (-167.0, 258.4)
- added H***: Val**, Via_016, F.Cu at (-168.3, 259.7)
- added H***: Val**, Via_016, F.Cu at (-170.2, 260.4)
- added H***: Val**, Via_016, F.Cu at (-172.1, 260.4)
- added H***: Val**, Via_016, F.Cu at (-174.0, 260.4)
- added PIN_ARRAY_3X1: Val**, PIN_ARRAY_3X1, F.Cu at (-214.6, 47.0)
- added PIN_ARRAY_3X1: Val**, PIN_ARRAY_3X1, F.Cu at (-214.6, 36.8)
- added PIN_ARRAY_3X1: Val**, PIN_ARRAY_3X1, F.Cu at (-242.6, 36.8)
- added PIN_ARRAY_3X1: Val**, PIN_ARRAY_3X1, F.Cu at (-242.6, 47.0)
- added PIN_ARRAY_3X1: Val**, PIN_ARRAY_3X1, F.Cu at (-168.9, 57.1)
- added PIN_ARRAY_3X1: Val**, PIN_ARRAY_3X1, F.Cu at (-168.9, 47.0)
- added PIN_ARRAY_3X1: Val**, PIN_ARRAY_3X1, F.Cu at (-141.0, 47.0)
- added PIN_ARRAY_3X1: Val**, PIN_ARRAY_3X1, F.Cu at (-141.0, 57.1)
- added PIN_ARRAY_5X1: Val**, PIN_ARRAY_5x1, F.Cu at (-228.6, 29.2)
- added PIN_ARRAY_5X1: Val**, PIN_ARRAY_5x1, F.Cu at (-154.9, 39.4)
- added PIN_ARRAY_5X1: Val**, PIN_ARRAY_5x1, F.Cu at (212.1, 365.8)
- added PIN_ARRAY_5X1: Val**, PIN_ARRAY_5x1, F.Cu at (233.7, 378.5)
- added PIN_ARRAY_5X1: Val**, PIN_ARRAY_5x1, F.Cu at (262.9, 365.8)
- added PIN_ARRAY_5X1: Val**, PIN_ARRAY_5x1, F.Cu at (284.5, 378.5)
- added PIN_ARRAY_5X1: Val**, PIN_ARRAY_5x1, F.Cu at (262.9, 459.7)
- added PIN_ARRAY_5X1: Val**, PIN_ARRAY_5x1, F.Cu at (241.3, 447.0)
- added PIN_ARRAY_5X1: Val**, PIN_ARRAY_5x1, F.Cu at (212.1, 459.7)
- added PIN_ARRAY_5X1: Val**, PIN_ARRAY_5x1, F.Cu at (190.5, 447.0)
- added R1: 1k, R_AXIAL_0W25_059A_PL, F.Cu at (-158.8, 240.7)
- added R1: 1k, R_AXIAL_0W25_059A_PL, F.Cu at (-223.5, 241.3)
- added R1: 1k, R_AXIAL_0W25_059A_PL, F.Cu at (-139.7, 118.1)
- added R2: 1k, R_AXIAL_0W25_059A_PL, F.Cu at (-137.2, 240.7)
- added R2: 1k, R_AXIAL_0W25_059A_PL, F.Cu at (-201.9, 241.3)
- added R2: 1k, R_AXIAL_0W25_059A_PL, F.Cu at (-118.1, 118.1)
- added R3: 6k8, R_AXIAL_0W25_059A_PL, F.Cu at (-133.3, 250.8)
- added R3: 6k8, R_AXIAL_0W25_059A_PL, F.Cu at (-198.1, 251.5)
- added R3: 6k8, R_AXIAL_0W25_059A_PL, F.Cu at (-114.3, 128.3)
- added U1: LM399, TO-46-PLASTIC, F.Cu at (-150.5, 265.4)
- added U1: LM399, TO-46-PLASTIC, F.Cu at (-215.3, 266.1)
- added U1: LM399, TO-46-PLASTIC, F.Cu at (-281.3, 266.1)
- added U1: LM399, TO-46-PLASTIC, F.Cu at (-281.3, 207.0)
- added U1: LM399, TO-46-PLASTIC, F.Cu at (-281.3, 144.1)
- added U1: LM399, TO-46-PLASTIC, F.Cu at (-130.8, 143.5)
- added U1: LM399, TO-46-PLASTIC, F.Cu at (-358.1, 143.5)
- added U2: OP07, DIP8_059A_PL, F.Cu at (-149.9, 249.6)
- added U2: OP07, DIP8_059A_PL, F.Cu at (-214.6, 250.2)
- added U2: OP07, DIP8_059A_PL, F.Cu at (-130.8, 127.0)
- moved U1 522.5 mm to (-207.0, 144.8), turned to 90 degrees
- moved G*** 260.0 mm to (59.7, 54.0)
Routing:
- net +VH: track 21.7 -> 533.6 mm
- net -VH: track 30.4 -> 509.3 mm
- net +VZ: track 24.5 -> 444.6 mm
- net -VZ: track 10.2 -> 409.6 mm
- net +VTOP: track 28.2 -> 0.00 mm
- net -VOP: track 25.6 -> 0.00 mm
- net N-0000011: track 13.5 -> 0.00 mm
- net +VOP: track 9.42 -> 0.00 mm
- added copper zone on B.Cu, net (none)
- removed copper zone on B.Cu, net GND
Other:
- board size 25.4 x 38.1 mm -> 767.1 x 471.2 mm
- copper layers 2 -> 4
- board text added: "AD584"
- board text added: "GND"
- board text added: "Vin"
- board text added: "Vout"
- board text added: "split middle designs"
- board text added: "upside down"

Commit message: old WIP
Parts:
- removed 4455-N2-5 (x32): Val**, 4455-N2-5
- removed the C1 at (-162.6, 245.7)
- removed the C1 at (-227.3, 246.4)
- removed the C1 at (-143.5, 123.2)
- removed the C2 at (-153.7, 245.7)
- removed the C2 at (-218.4, 246.4)
- removed the C2 at (-134.6, 123.2)
- removed the C3 at (-129.5, 245.7)
- removed the C3 at (-194.3, 246.4)
- removed the C3 at (-110.5, 123.2)
- removed the H*** at (-174.0, 237.5)
- removed the H*** at (-261.0, 257.2)
- removed the H*** at (-174.0, 262.3)
- removed the H*** at (-174.0, 264.2)
- removed the H*** at (-174.0, 266.1)
- removed the H*** at (-174.0, 268.0)
- removed the H*** at (-174.0, 269.9)
- removed the H*** at (-174.0, 271.8)
- removed the H*** at (-174.0, 273.7)
- removed the H*** at (-173.4, 275.0)
- removed the H*** at (-172.7, 276.2)
- removed the H*** at (-171.4, 276.9)
- removed the H*** at (-301.6, 234.3)
- removed the H*** at (-170.2, 277.5)
- removed the H*** at (-168.3, 277.5)
- removed the H*** at (-166.4, 277.5)
- removed the H*** at (-164.5, 277.5)
- removed the H*** at (-162.6, 277.5)
- removed the H*** at (-160.7, 277.5)
- removed the H*** at (-158.8, 277.5)
- removed the H*** at (-156.8, 277.5)
- removed the H*** at (-154.9, 277.5)
- removed the H*** at (-153.0, 277.5)
- removed the H*** at (-261.0, 234.3)
- removed the H*** at (-151.3, 277.5)
- removed the H*** at (-149.7, 277.5)
- removed the H*** at (-148.0, 277.5)
- removed the H*** at (-146.1, 277.5)
- removed the H*** at (-144.1, 277.5)
- removed the H*** at (-142.2, 277.5)
- removed the H*** at (-140.3, 277.5)
- removed the H*** at (-138.4, 277.5)
- removed the H*** at (-136.5, 277.5)
- removed the H*** at (-134.6, 277.5)
- removed the H*** at (-301.6, 257.2)
- removed the H*** at (-132.7, 277.5)
- removed the H*** at (-130.8, 277.5)
- removed the H*** at (-129.5, 276.9)
- removed the H*** at (-127.6, 275.0)
- removed the H*** at (-127.0, 273.7)
- removed the H*** at (-128.3, 276.2)
- removed the H*** at (-127.0, 271.8)
- removed the H*** at (-127.0, 269.9)
- removed the H*** at (-127.0, 268.0)
- removed the H*** at (-127.0, 266.1)
- removed the H*** at (-301.6, 198.1)
- removed the H*** at (-127.0, 264.2)
- removed the H*** at (-127.0, 262.3)
- removed the H*** at (-127.0, 260.4)
- removed the H*** at (-127.0, 252.7)
- removed the H*** at (-127.0, 250.8)
- removed the H*** at (-127.0, 248.9)
- removed the H*** at (-127.0, 247.0)
- removed the H*** at (-127.0, 245.1)
- removed the H*** at (-127.0, 243.2)
- removed the H*** at (-127.0, 241.3)
- removed the H*** at (-261.0, 175.3)
- removed the H*** at (-127.0, 239.4)
- removed the H*** at (-127.0, 237.5)
- removed the H*** at (-128.9, 237.5)
- removed the H*** at (-130.8, 237.5)
- removed the H*** at (-134.0, 234.3)
- removed the H*** at (-134.0, 230.5)
- removed the H*** at (-134.0, 232.4)
- removed the H*** at (-134.0, 236.2)
- removed the H*** at (-132.7, 237.5)
- removed the H*** at (-135.9, 230.5)
- removed the H*** at (-301.6, 175.3)
- removed the H*** at (-137.8, 230.5)
- removed the H*** at (-139.7, 230.5)
- removed the H*** at (-141.6, 230.5)
- removed the H*** at (-143.5, 230.5)
- removed the H*** at (-145.4, 230.5)
- removed the H*** at (-147.3, 230.5)
- removed the H*** at (-149.2, 230.5)
- removed the H*** at (-151.8, 230.5)
- removed the H*** at (-153.7, 230.5)
- removed the H*** at (-155.6, 230.5)
- removed the H*** at (-261.0, 198.1)
- removed the H*** at (-157.5, 230.5)
- removed the H*** at (-159.4, 230.5)
- removed the H*** at (-161.3, 230.5)
- removed the H*** at (-163.2, 230.5)
- removed the H*** at (-167.0, 230.5)
- removed the H*** at (-165.1, 230.5)
- removed the H*** at (-128.9, 252.7)
- removed the H*** at (-128.9, 260.4)
- removed the H*** at (-130.8, 260.4)
- removed the H*** at (-130.8, 252.7)
- removed the H*** at (-261.0, 135.3)
- removed the H*** at (-134.0, 256.5)
- removed the H*** at (-134.0, 254.6)
- removed the H*** at (-134.0, 258.4)
- removed the H*** at (-132.7, 259.7)
- removed the H*** at (-132.7, 253.4)
- removed the H*** at (-167.0, 232.4)
- removed the H*** at (-167.0, 234.3)
- removed the H*** at (-172.1, 237.5)
- removed the H*** at (-170.2, 237.5)
- removed the H*** at (-168.3, 237.5)
- removed the H*** at (-301.6, 112.4)
- removed the H*** at (-167.0, 236.2)
- removed the H*** at (-137.8, 271.8)
- removed the H*** at (-135.9, 269.2)
- removed the H*** at (-134.6, 270.5)
- removed the H*** at (-135.9, 271.8)
- removed the H*** at (-139.7, 271.1)
- removed the H*** at (-142.2, 266.7)
- removed the H*** at (-137.8, 268.6)
- removed the H*** at (-139.1, 267.3)
- removed the H*** at (-139.7, 265.4)
- removed the H*** at (-130.2, 256.5)
- removed the H*** at (-261.0, 112.4)
- removed the H*** at (-141.0, 269.9)
- removed the H*** at (-141.6, 268.6)
- removed the H*** at (-139.7, 263.5)
- removed the H*** at (-139.7, 261.6)
- removed the H*** at (-140.3, 259.7)
- removed the H*** at (-141.6, 258.4)
- removed the H*** at (-142.9, 257.2)
- removed the H*** at (-144.1, 255.9)
- removed the H*** at (-146.1, 255.3)
- removed the H*** at (-148.0, 254.6)
- removed the H*** at (-301.6, 135.3)
- removed the H*** at (-149.7, 254.6)
- removed the H*** at (-151.3, 254.6)
- removed the H*** at (-153.7, 255.3)
- removed the H*** at (-155.6, 255.3)
- removed the H*** at (-110.5, 134.6)
- removed the H*** at (-151.1, 111.8)
- removed the H*** at (-110.5, 111.8)
- removed the H*** at (-151.1, 134.6)
- removed the H*** at (-337.8, 134.6)
- removed the H*** at (-378.5, 111.8)
- removed the H*** at (-337.8, 111.8)
- removed the H*** at (-378.5, 134.6)
- removed the H*** at (-170.8, 233.7)
- removed the H*** at (-227.3, 135.9)
- removed the H*** at (-186.7, 113.0)
- removed the H*** at (-227.3, 113.0)
- removed the H*** at (-186.7, 135.9)
- removed the H*** at (-248.9, 38.1)
- removed the H*** at (-208.3, 15.2)
- removed the H*** at (-248.9, 15.2)
- removed the H*** at (-208.3, 38.1)
- removed the H*** at (-45.7, 54.6)
- removed the H*** at (-86.4, 31.8)
- removed the H*** at (-130.2, 233.7)
- removed the H*** at (-45.7, 31.8)
- removed the H*** at (-86.4, 54.6)
- removed the H*** at (283.2, 435.6)
- removed the H*** at (191.8, 458.5)
- removed the H*** at (232.4, 435.6)
- removed the H*** at (191.8, 435.6)
- removed the H*** at (232.4, 458.5)
- removed the H*** at (242.6, 458.5)
- removed the H*** at (242.6, 435.6)
- removed the H*** at (283.2, 458.5)
- removed the H*** at (-170.8, 256.5)
- removed the H*** at (232.4, 367.0)
- removed the H*** at (191.8, 389.9)
- removed the H*** at (232.4, 389.9)
- removed the H*** at (191.8, 367.0)
- removed the H*** at (242.6, 367.0)
- removed the H*** at (283.2, 389.9)
- removed the H*** at (242.6, 389.9)
- removed the H*** at (283.2, 367.0)
- removed the H*** at (141.0, 369.6)
- removed the H*** at (100.3, 392.4)
- removed the H*** at (-235.6, 257.2)
- removed the H*** at (141.0, 392.4)
- removed the H*** at (100.3, 369.6)
- removed the H*** at (49.5, 369.6)
- removed the H*** at (90.2, 392.4)
- removed the H*** at (49.5, 392.4)
- removed the H*** at (90.2, 369.6)
- removed the H*** at (141.0, 461.0)
- removed the H*** at (100.3, 438.1)
- removed the H*** at (141.0, 438.1)
- removed the H*** at (100.3, 461.0)
- removed the H*** at (-194.9, 234.3)
- removed the H*** at (90.2, 461.0)
- removed the H*** at (49.5, 438.1)
- removed the H*** at (90.2, 438.1)
- removed the H*** at (49.5, 461.0)
- removed the H*** at (379.7, 463.6)
- removed the H*** at (339.1, 440.7)
- removed the H*** at (379.7, 440.7)
- removed the H*** at (339.1, 463.6)
- removed the H*** at (340.4, 387.4)
- removed the H*** at (381.0, 364.5)
- removed the H*** at (-235.6, 234.3)
- removed the H*** at (340.4, 364.5)
- removed the H*** at (381.0, 387.4)
- removed the H*** at (-174.0, 239.4)
- removed the H*** at (-174.0, 241.3)
- removed the H*** at (-174.0, 243.2)
- removed the H*** at (-174.0, 245.1)
- removed the H*** at (-174.0, 247.0)
- removed the H*** at (-174.0, 248.9)
- removed the H*** at (-174.0, 250.8)
- removed the H*** at (-174.0, 252.7)
- removed the H*** at (-194.9, 257.2)
- removed the H*** at (-172.1, 252.7)
- removed the H*** at (-170.2, 252.7)
- removed the H*** at (-168.3, 253.4)
- removed the H*** at (-167.0, 254.6)
- removed the H*** at (-167.0, 256.5)
- removed the H*** at (-167.0, 258.4)
- removed the H*** at (-168.3, 259.7)
- removed the H*** at (-170.2, 260.4)
- removed the H*** at (-172.1, 260.4)
- removed the H*** at (-174.0, 260.4)
- removed PIN_ARRAY_3X1 (x8): Val**, PIN_ARRAY_3X1
- removed PIN_ARRAY_5X1 (x10): Val**, PIN_ARRAY_5x1
- removed the R1 at (-158.8, 240.7)
- removed the R1 at (-223.5, 241.3)
- removed the R1 at (-139.7, 118.1)
- removed the R2 at (-137.2, 240.7)
- removed the R2 at (-201.9, 241.3)
- removed the R2 at (-118.1, 118.1)
- removed the R3 at (-133.3, 250.8)
- removed the R3 at (-198.1, 251.5)
- removed the R3 at (-114.3, 128.3)
- removed the U1 at (-150.5, 265.4)
- removed the U1 at (-215.3, 266.1)
- removed the U1 at (-281.3, 266.1)
- removed the U1 at (-281.3, 207.0)
- removed the U1 at (-281.3, 144.1)
- removed the U1 at (-130.8, 143.5)
- removed the U1 at (-358.1, 143.5)
- removed the U1 at (-207.0, 144.8)
- removed the U2 at (-149.9, 249.6)
- removed the U2 at (-214.6, 250.2)
- removed the U2 at (-130.8, 127.0)
- added C1: 0.1uF, CERCAP_2_059A, F.Cu at (196.8, 134.6)
- added C2: 0.1uF, CERCAP_2_059A, F.Cu at (195.6, 146.1)
- added C3: 10nF, CERCAP_2_059A, F.Cu at (180.3, 146.1)
- added H***: Val**, hole_M3_2, F.Cu at (167.6, 133.3)
- added H***: Val**, hole_M3_2, F.Cu at (208.3, 133.3)
- added H***: Val**, hole_M3_2, F.Cu at (208.3, 174.0)
- added H***: Val**, hole_M3_2, F.Cu at (167.6, 174.0)
- added P1: CONN_5X1, 4455-N2-5, F.Cu at (188.0, 135.9)
- added R1: 1k, R_AXIAL_0W25_059A_PL, F.Cu at (198.1, 141.0)
- added R2: 1k, R_AXIAL_0W25_059A_PL, F.Cu at (177.8, 141.0)
- added R3: 6k8, R_AXIAL_0W25_059A_PL, F.Cu at (175.3, 151.1)
- added U1: LM399A, TO-46-PLASTIC, F.Cu at (188.0, 165.1)
- added U2: OP07, DIP8_059A_PL, F.Cu at (184.2, 149.9)
Routing:
- net +VH: track 533.6 -> 0.00 mm
- net -VH: track 509.3 -> 0.00 mm
- net +VZ: track 444.6 -> 0.00 mm
- net -VZ: track 409.6 -> 0.00 mm
- net -Vref: track 0.00 -> 160.4 mm
- net 15V: track 0.00 -> 77.4 mm
- net +Vref: track 0.00 -> 70.2 mm
- net N-000006: track 0.00 -> 25.0 mm
- net N-000007: track 0.00 -> 15.5 mm
- removed copper zone on B.Cu, net (none)
Other:
- board size 767.1 x 471.2 mm -> 48.3 x 48.3 mm
- board text removed: "AD584"
- board text removed: "GND"
- board text removed: "Vin"
- board text removed: "Vout"
- board text removed: "split middle designs"
- board text removed: "upside down"
