File: kicad/lm399-stick.kicad_pcb (KiCad board)
At the start: 4 copper layers, 48.3 x 16.5 mm, 18 parts, among them P1 CONN_1X1, P2 CONN_1X1, P3 CONN_1X1, P4 CONN_1X1, P5 CONN_2X1, U1 LM399A, U2 OP07

Commit message: v1.1
Parts:
- removed the H*** at (209.6, 137.2)
- removed the H*** at (209.6, 149.9)
- added H***: Val**, 1pin_056_079, F.Cu at (209.6, 137.2)
- added H***: Val**, 1pin_056_079, F.Cu at (209.6, 149.9)
- P1, P2, P3, P4: footprint 1pin_060_079 -> 1pin_056_079
Changed lines of the file:
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@@
     (links 25)
     (no_connects 0)
-    (area 160.203445 133.731 212.753222 153.289)
+    (area 163.144999 135.204999 211.505001 151.815001)
     (thickness 1.6)
     (drawings 32)
@@
     (mod_text_width 0.15)
     (pad_size 2.0066 2.0066)
-    (pad_drill 1.524)
+    (pad_drill 1.4224)
     (pad_to_mask_clearance 0)
     (aux_axis_origin 0 0)
@@
       (xy -0.90932 1.3462)) (layer F.SilkS) (width 0.00254))
   )
-  (module 1pin_060_079 (layer F.Cu)
+  (module 1pin_056_079 (layer F.Cu)
+    (at 165.1 137.16)
+    (descr "1 pin, 0.056\" drill, 0.079\" round pad")
+    (fp_text reference P2 (at 0 -2.54) (layer F.SilkS) hide
+      (effects (font (size 1.016 1.016) (thickness 0.254)))
+    )
+    (fp_text value CONN_1X1 (at 0 2.54) (layer F.SilkS) hide
+      (effects (font (size 1.016 1.016) (thickness 0.254)))
+    )
+    (pad 1 thru_hole circle (at 0 0) (size 2.0066 2.0066) (drill 1.4224)
+      (layers *.Cu *.Mask F.SilkS)
+      (net 2 -Vz)
+    )
+  )
+  (module 1pin_056_079 (layer F.Cu)
     (at 209.55 137.16)
-    (descr "1 pin, 0.060\" drill, 0.079\" round pad")
+    (descr "1 pin, 0.056\" drill, 0.079\" round pad")
     (path 1pin)
     (fp_text reference H*** (at 0 -2.54) (layer F.SilkS) hide
@@
       (effects (font (size 1.016 1.016) (thickness 0.254)))
     )
-    (pad 1 thru_hole circle (at 0 0) (size 2.0066 2.0066) (drill 1.524)
-      (layers *.Cu *.Mask F.SilkS)
-    )
-  )
-  (module 1pin_060_079 (layer F.Cu)
+    (pad 1 thru_hole circle (at 0 0) (size 2.0066 2.0066) (drill 1.4224)
+      (layers *.Cu *.Mask F.SilkS)
+    )
+  )
+  (module 1pin_056_079 (layer F.Cu)
     (at 209.55 149.86)
-    (descr "1 pin, 0.060\" drill, 0.079\" round pad")
+    (descr "1 pin, 0.056\" drill, 0.079\" round pad")
     (path 1pin)
     (fp_text reference H*** (at 0 -2.54) (layer F.SilkS) hide
@@
       (effects (font (size 1.016 1.016) (thickness 0.254)))
     )
-    (pad 1 thru_hole circle (at 0 0) (size 2.0066 2.0066) (drill 1.524)
-      (layers *.Cu *.Mask F.SilkS)
-    )
-  )
-  (module 1pin_060_079 (layer F.Cu)
+    (pad 1 thru_hole circle (at 0 0) (size 2.0066 2.0066) (drill 1.4224)
+      (layers *.Cu *.Mask F.SilkS)
+    )
+  )
+  (module 1pin_056_079 (layer F.Cu)
     (at 165.1 149.86)
-    (descr "1 pin, 0.060\" drill, 0.079\" round pad")
+    (descr "1 pin, 0.056\" drill, 0.079\" round pad")
     (fp_text reference P1 (at 0 -2.54) (layer F.SilkS) hide
       (effects (font (size 1.016 1.016) (thickness 0.254)))
@@
       (effects (font (size 1.016 1.016) (thickness 0.254)))
     )
-    (pad 1 thru_hole rect (at 0 0) (size 2.0066 2.0066) (drill 1.524)
+    (pad 1 thru_hole rect (at 0 0) (size 2.0066 2.0066) (drill 1.4224)
       (layers *.Cu *.Mask F.SilkS)
       (net 6 Vcc)
     )
   )
-  (module 1pin_060_079 (layer F.Cu)
-    (at 165.1 137.16)
-    (descr "1 pin, 0.060\" drill, 0.079\" round pad")
-    (fp_text reference P2 (at 0 -2.54) (layer F.SilkS) hide
+  (module 1pin_056_079 (layer F.Cu)
+    (at 187.96 142.24)
+    (descr "1 pin, 0.056\" drill, 0.079\" round pad")
+    (fp_text reference P4 (at 0 -2.54) (layer F.SilkS) hide
       (effects (font (size 1.016 1.016) (thickness 0.254)))
     )
@@
       (effects (font (size 1.016 1.016) (thickness 0.254)))
     )
-    (pad 1 thru_hole circle (at 0 0) (size 2.0066 2.0066) (drill 1.524)
-      (layers *.Cu *.Mask F.SilkS)
-      (net 2 -Vz)
-    )
-  )
-  (module 1pin_060_079 (layer F.Cu)
-    (at 187.96 142.24)
-    (descr "1 pin, 0.060\" drill, 0.079\" round pad")
-    (fp_text reference P4 (at 0 -2.54) (layer F.SilkS) hide
+    (pad 1 thru_hole circle (at 0 0) (size 2.0066 2.0066) (drill 1.4224)
+      (layers *.Cu *.Mask F.SilkS)
+      (net 2 -Vz)
+    )
+  )
+  (module 1pin_056_079 (layer F.Cu)
+    (at 187.96 144.78)
+    (descr "1 pin, 0.056\" drill, 0.079\" round pad")
+    (fp_text reference P3 (at 0 -2.54) (layer F.SilkS) hide
       (effects (font (size 1.016 1.016) (thickness 0.254)))
     )
@@
       (effects (font (size 1.016 1.016) (thickness 0.254)))
     )
-    (pad 1 thru_hole circle (at 0 0) (size 2.0066 2.0066) (drill 1.524)
-      (layers *.Cu *.Mask F.SilkS)
-      (net 2 -Vz)
-    )
-  )
-  (module 1pin_060_079 (layer F.Cu)
-    (at 187.96 144.78)
-    (descr "1 pin, 0.060\" drill, 0.079\" round pad")
-    (fp_text reference P3 (at 0 -2.54) (layer F.SilkS) hide
-      (effects (font (size 1.016 1.016) (thickness 0.254)))
-    )
-    (fp_text value CONN_1X1 (at 0 2.54) (layer F.SilkS) hide
-      (effects (font (size 1.016 1.016) (thickness 0.254)))
-    )
-    (pad 1 thru_hole rect (at 0 0) (size 2.0066 2.0066) (drill 1.524)
+    (pad 1 thru_hole rect (at 0 0) (size 2.0066 2.0066) (drill 1.4224)
       (layers *.Cu *.Mask F.SilkS)
       (net 1 +Vz)

Commit message: v1.2
Parts:
- removed H*** (x2): Val**, 1pin_056_079
- added D1: 1N4148, DIODE_SS_059A_03_PL, F.Cu at (185.4, 144.8)
- added R5: 470k, R_AXIAL_0W25_V_059A_PL, F.Cu at (182.9, 141.0)
- R4: value 200k -> 1M; footprint R_AXIAL_0W25_059A_PL -> R_AXIAL_0W25_V_059A_PL
- moved C2 13.0 mm to (194.3, 137.2)
- moved P5 12.8 mm to (184.2, 137.2)
- moved R1 5.68 mm to (188.0, 139.7), turned to 0 degrees
- moved P3 5.68 mm to (193.0, 147.3)
- moved P4 5.68 mm to (193.0, 144.8)
- moved G*** 4.49 mm to (196.8, 143.5)
- moved C1 4.26 mm to (189.2, 147.3)
- moved R4 2.84 mm to (182.9, 148.6)
- moved R2 2.54 mm to (170.2, 138.4)
- moved R3 2.54 mm to (167.6, 148.6)
- moved U1 2.54 mm to (206.4, 141.6)
- moved U2 1.27 mm to (180.3, 146.1)
- turned C4 to 90 degrees
Connections:
- C4 pad 1: N-000004 -> N-000006
- C4 pad 2: N-000007 -> -Vz
- R1 pad 1: N-000004 -> N-000007
- R2 pad 1: N-000004 -> N-000007
- R2 pad 2: N-000007 -> N-000006
- R3 pad 1: N-000007 -> N-000006
- R4 pad 2: +Vz -> N-000001
- U2 pad 2: N-000007 -> N-000006
- U2 pad 6: N-000004 -> N-000007
Routing:
- net Vcc: track 31.1 -> 60.8 mm
- net -Vz: track 131.7 -> 153.6 mm
- net N-000004: track 20.4 -> 0.00 mm
- net N-000006: track 0.00 -> 20.3 mm
- net +Vz: track 63.8 -> 52.4 mm
- net N-000001: track 0.00 -> 6.13 mm
- net N-000007: track 23.7 -> 19.4 mm
- net N-000009: track 23.7 -> 28.0 mm
Other:
- board size 48.3 x 16.5 mm -> 49.5 x 16.5 mm
- board text added: "10 to 18V"
- board text added: "HEATR"
- board text added: "github.com/ pepaslabs/ lm399-stick"
- board text added: "v1.2"
- board text removed: "HEATER"
- board text removed: "github.com/pepaslabs/lm399-stick"
- board text removed: "v1.1"

Commit message: v1.3
Parts:
- removed D1: 1N4148, DIODE_SS_059A_03_PL
- removed the G*** at (196.8, 143.5)
- removed R4: 1M, R_AXIAL_0W25_V_059A_PL
- removed R5: 470k, R_AXIAL_0W25_V_059A_PL
- added G***: OSHW-logo_silkscreen-front_4mm, OSHW-logo_silkscreen-front_4mm, F.Cu at (192.4, 143.5)
- R2: value 1k -> 3k3
- R3: value 6k8 -> 22k
- moved C1 6.35 mm to (182.9, 147.3), turned to 270 degrees
- moved P3 5.68 mm to (188.0, 144.8)
- moved P4 5.68 mm to (188.0, 147.3)
- moved R1 5.08 mm to (182.9, 139.7)
- moved U1 3.81 mm to (202.6, 141.6)
- moved C2 3.18 mm to (191.1, 137.2)
- moved P5 1.27 mm to (182.9, 137.2)
Routing:
- net -Vz: track 153.6 -> 123.5 mm
- net Vcc: track 60.8 -> 49.1 mm
- net N-000002: track 28.0 -> 37.6 mm
- net +Vz: track 52.4 -> 45.6 mm
- net N-000001: track 6.13 -> 0.00 mm
- net N-000008: track 19.4 -> 14.3 mm
Other:
- board size 49.5 x 16.5 mm -> 45.7 x 16.5 mm
- board text added: "v1.3"
- board text removed: "v1.2"
